File: Input-Protection.kicad_pcb (KiCad board)
At the start: 2 copper layers, 80 x 50 mm, 77 parts, among them J101 KLDX-0202-B, J102 EBWA-02-B, J103 EBWA-02-B, J104 KLDX-0202-B, Q201 MCU18P10Y-TP, Q601 BC846, Q602 MCU18P10Y-TP, U401 LM4040N-5.0, U501 LM393, U502 LM393, U503 INA169NA/3K

Commit message: feat: revision B release
Parts:
- FID901, FID902, FID903: footprint Fiducial:Fiducial_Cross_0.5mm_Mask2mm -> Fiducial:Fiducial_1mm_Mask2mm
Routing:
- net Net-(U501B-+): track 14.2 -> 18.3 mm
- net VCC_5V: track 100.6 -> 96.6 mm
- net /ARCHITECTURE/5. COMPARATOR/~{OC_DETECT}: track 21.3 -> 23.8 mm
- net /ARCHITECTURE/2. POLARITY PROTECTION/VPROT: track 21.6 -> 22.6 mm
Other:
- board text added: "0.02mm"
- board text added: "0.035mm (1.00oz)"
- board text added: "1.48mm"
- board text added: "ALL DIMENSIONS IN MILLIMETERS UNLESS OTHERWISE SPECIFIED."
- board text added: "B"
- board text added: "B.Mask"
- board text added: "B.Paste"
- board text added: "B.Silkscreen"
- board text added: "BOTTOM VIEW"
- board text added: "COMPONENTS"
- board text added: "Copper"
- board text added: "Core"
- board text added: "DRILL TABLE"
- board text added: "Dielectric"
- board text added: "Direct Printing"
- board text added: "F.Mask"
- board text added: "F.Paste"
- board text added: "F.Silkscreen"
- board text added: "FR4_7628"
- board text added: "GBR"
- board text added: "Gerber"
- board text added: "L1 (Sig, PWR)"
- board text added: "L2 (Sig, GND)"
- board text added: "LAYER STACKUP LEGEND"
- board text added: "Layer"
- board text added: "Legend"
- board text added: "Material"
- board text added: "Note: external layer thicknesses are specified after plating"
- board text added: "Paste Mask"
- board text added: "Plane"
- board text added: "Signal"
- board text added: "Solder Mask"
- board text added: "Solder Resist"
- board text added: "TOP VIEW"
- board text added: "Thickness"
- board text added: "Total thickness: 1.59mm"
- board text added: "Type"
- board text removed: "A"
- board text removed: "Bottom View"
- board text removed: "Components"
- board text removed: "Drill Table"
- board text removed: "Layer Stack Legend"
- board text removed: "Top View"
