File: Miscellaneous.kicad_sch (KiCad schematic)
At the start: 8 parts

Commit message: feat: revision B release
Parts:
- FID901, FID902, FID903: footprint Fiducial:Fiducial_Cross_0.5mm_Mask2mm -> Fiducial:Fiducial_1mm_Mask2mm
Changed lines of the file:
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@@
 			)
 		)
-		(property "Footprint" "Fiducial:Fiducial_Cross_0.5mm_Mask2mm"
+		(property "Footprint" "Fiducial:Fiducial_1mm_Mask2mm"
 			(at 139.7 52.07 0)
 			(effects
@@
 			)
 		)
-		(property "Footprint" "Fiducial:Fiducial_Cross_0.5mm_Mask2mm"
+		(property "Footprint" "Fiducial:Fiducial_1mm_Mask2mm"
 			(at 139.7 59.69 0)
 			(effects
@@
 			)
 		)
-		(property "Footprint" "Fiducial:Fiducial_Cross_0.5mm_Mask2mm"
+		(property "Footprint" "Fiducial:Fiducial_1mm_Mask2mm"
 			(at 139.7 67.31 0)
 			(effects
