File: Revision History.kicad_sch (KiCad schematic)
At the start: 0 parts

Commit message: fix: template changes
Changed lines of the file:
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@@
 		(exclude_from_sim no)
 		(at 220.98 35.56 0)
-		(size 58.42 111.76)
+		(size 58.42 97.79)
 		(margins 1.4287 1.4287 1.4287 1.4287)
 		(stroke
@@
 	(text_box "[${#}] ${TITLE}"
 		(exclude_from_sim no)
-		(at 80.01 16.51 0)
+		(at 82.55 15.24 0)
 		(size 137.16 12.7)
 		(margins 4.4999 4.4999 4.4999 4.4999)
@@
 		(effects
 			(font
-				(face "Times New Roman")
 				(size 6 6)
 				(thickness 1.2)
@@
 	(text_box "${RELEASE_BODY_1.0.0}"
 		(exclude_from_sim no)
-		(at 22.86 35.56 0)
-		(size 58.42 146.05)
+		(at 25.4 35.56 0)
+		(size 55.88 146.05)
 		(margins 1.4287 1.4287 1.4287 1.4287)
 		(stroke
@@
 		(exclude_from_sim no)
 		(at 154.94 35.56 0)
-		(size 58.42 111.76)
+		(size 58.42 97.79)
 		(margins 1.4287 1.4287 1.4287 1.4287)
 		(stroke
@@
 		(exclude_from_sim no)
 		(at 88.9 35.56 0)
-		(size 57.15 105.41)
+		(size 57.15 97.79)
 		(margins 1.4287 1.4287 1.4287 1.4287)
 		(stroke
@@
 	(text_box "${RELEASE_TITLE_1.0.0}"
 		(exclude_from_sim no)
-		(at 20.32 31.75 0)
-		(size 57.15 7.62)
+		(at 24.13 31.75 0)
+		(size 53.34 7.62)
 		(margins 1.4287 1.4287 1.4287 1.4287)
 		(stroke
@@
 	(polyline
 		(pts
-			(xy 85.09 31.75) (xy 85.09 149.86)
+			(xy 85.09 31.75) (xy 85.09 190.5)
 		)
 		(stroke
@@
 	(polyline
 		(pts
-			(xy 151.13 31.75) (xy 151.13 149.86)
+			(xy 151.13 31.75) (xy 151.13 133.35)
 		)
 		(stroke
@@
 	(polyline
 		(pts
-			(xy 19.05 31.75) (xy 19.05 190.5)
+			(xy 21.59 31.75) (xy 21.59 190.5)
 		)
 		(stroke
@@
 	(polyline
 		(pts
-			(xy 217.17 31.75) (xy 217.17 149.86)
-		)
-		(stroke
+			(xy 217.17 31.75) (xy 217.17 133.35)
+		)
+		(stroke

Commit message: feat: revision B release
Changed lines of the file:
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@@
 		)
 	)
-	(text_box "${RELEASE_BODY_1.0.1}"
+	(text_box "${RELEASE_BODY_1.1.0}"
 		(exclude_from_sim no)
 		(at 88.9 35.56 0)
@@
 		)
 	)
-	(text_box "${RELEASE_TITLE_1.0.1}"
+	(text_box "${RELEASE_TITLE_1.1.0}"
 		(exclude_from_sim no)
 		(at 86.36 31.75 0)
